Commit message: Update hardware xacro configuration

File: src/erob_description/urdf/erob_hardware.urdf.xacro (robot description, xacro)
@@ -4,3 +4,4 @@
   <xacro:include filename="$(find erob_description)/urdf/erob_real.ros2_control.xacro" />
   <xacro:erob_real_ros2_control name="RealLeftArm" />
+  <xacro:erob_mock_ros2_control name="MockRightArmAndHead" />
 </robot>

File: src/erob_description/urdf/erob_real.ros2_control.xacro (robot description, xacro)
@@ -36,3 +36,46 @@
     </ros2_control>
   </xacro:macro>
+  <xacro:macro name="erob_mock_ros2_control" params="name">
+    <ros2_control name="${name}" type="system">
+      <hardware>
+        <plugin>mock_components/GenericSystem</plugin>
+      </hardware>
+      <joint name="R_Joint_1">
+        <command_interface name="position" />
+        <state_interface name="position" />
+      </joint>
+      <joint name="R_Joint_2">
+        <command_interface name="position" />
+        <state_interface name="position" />
+      </joint>
+      <joint name="R_Joint_3">
+        <command_interface name="position" />
+        <state_interface name="position" />
+      </joint>
+      <joint name="R_Joint_4">
+        <command_interface name="position" />
+        <state_interface name="position" />
+      </joint>
+      <joint name="R_Joint_5">
+        <command_interface name="position" />
+        <state_interface name="position" />
+      </joint>
+      <joint name="R_Joint_6">
+        <command_interface name="position" />
+        <state_interface name="position" />
+      </joint>
+      <joint name="R_Joint_7">
+        <command_interface name="position" />
+        <state_interface name="position" />
+      </joint>
+      <joint name="neck_joint">
+        <command_interface name="position" />
+        <state_interface name="position" />
+      </joint>
+      <joint name="head_joint">
+        <command_interface name="position" />
+        <state_interface name="position" />
+      </joint>
+    </ros2_control>
+  </xacro:macro>
 </robot>
